File: pcb/gas-sensor/gas-sensor.kicad_sch (KiCad schematic)
At the start: 7 parts

Commit message: initial schematic
Parts:
- removed J? (x2): Conn_01x07, symbol Connector_Generic:Conn_01x07
- added C1, C2: 100nF, Capacitor_SMD:C_0603_1608Metric, symbol Device:C_Small
- added D1: D_Small, Diode_SMD:D_0603_1608Metric, symbol Device:D_Small
- added J1: MicroLab Input, Connector_PinSocket_2.54mm:PinSocket_2x06_P2.54mm_Vertical, symbol Connector_Generic:Conn_02x06_Odd_Even
- added Q1, Q2, Q3, Q4: T2N7002AK, Package_TO_SOT_SMD:SOT-23, symbol Transistor_FET:BSS138
- added R1, R2, R3, R4, R5, R6, R7, R8: 10k, Resistor_SMD:R_0603_1608Metric, symbol Device:R_Small
- added U3, U4: XC9265A331MR-G, SamacSys:SOT95P280X130-5N, symbol SamacSys:XC9265A331MR-G
- J2: renamed from J?; value Conn_01x02 -> Pump; footprint (none) -> Connector_PinSocket_2.54mm:PinSocket_1x02_P2.54mm_Vertical
- J3: renamed from J?; value Conn_01x04 -> DFRobot O2; footprint (none) -> Connector_PinSocket_2.54mm:PinSocket_1x04_P2.54mm_Vertical
- J4: renamed from J?; value Conn_01x04 -> DFRobot NH3; footprint (none) -> Connector_PinSocket_2.54mm:PinSocket_1x04_P2.54mm_Vertical
- U1: renamed from U?; value USEQGSE -> USEQGSE CO2
- U2: renamed from U?; value USEQGSE -> USEQGSE CH4
Connections:
- net SDA: now reaches J3.1 (Pin_1)
- net SDA: now also J4.1 (Pin_1), J1.1 (Pin_1), Q1.3 (D), Q3.3 (D), R2.2, R6.2
- net SCL: now reaches J3.2 (Pin_2)
- net SCL: now also J4.2 (Pin_2), J1.3 (Pin_3), Q2.3 (D), Q4.3 (D), R4.1, R8.1
- net GND: now reaches J3.3 (Pin_3)
- net GND: now also J2.2 (Pin_2), J4.3 (Pin_3), U1.17 (GND), U1.19 (GND), U1.28 (GND), U1.29 (GND), U1.30 (GND), U1.5 (GND), U1.7 (GND), U2.17 (GND), U2.19 (GND), U2.28 (GND), U2.29 (GND), U2.30 (GND), U2.5 (GND), U2.7 (GND), C1.1, C2.1, D1.2 (A), J1.7 (Pin_7), U3.2 (GND), U4.2 (GND)
- net V_O2: now reaches J3.4 (Pin_4)
- net V_O2: now also J1.4 (Pin_4)
- net V_CH4: now reaches U2.1 (VCC)
- net V_CH4: now also U2.23 (CS), Q3.1 (G), Q4.1 (G), R5.1, R7.2, U4.4 (VOUT)
- net CH4_INT: now reaches U2.25 (INT)
- net CH4_INT: now also J1.11 (Pin_11)
- net at U2.26 (SDA): now also Q3.2 (S), R5.2
- net at U2.3 (CAP): now also C2.2
- net at U2.37 (SCL): now also Q4.2 (S), R7.1
- net V_PUMP: now reaches J2.1 (Pin_1)
- net V_PUMP: now also D1.1 (K), J1.8 (Pin_8)
- net V_NH3: now reaches J4.4 (Pin_4)
- net V_NH3: now also J1.6 (Pin_6)
- net V_CO2: now reaches U1.1 (VCC)
- net V_CO2: now also U1.23 (CS), Q1.1 (G), Q2.1 (G), R1.1, R3.2, U3.4 (VOUT)
- net CO2_INT: now reaches U1.25 (INT)
- net CO2_INT: now also J1.9 (Pin_9)
- net at U1.26 (SDA): now also Q1.2 (S), R1.2
- net at U1.3 (CAP): now also C1.2
- net at U1.37 (SCL): now also Q2.2 (S), R3.1
- new net: J1.10 (Pin_10), U3.1 (VIN), U3.3 (CE)
- new net: J1.12 (Pin_12), U4.1 (VIN), U4.3 (CE)
- new net VCC: J1.5 (Pin_5), R2.1, R4.2, R6.1, R8.2
- no-connect marks 0 -> 7
Other:
- moved on the sheet: J2, J3, J4, U1, U2
