File: pcb/pcb_middle/pcb_middle.kicad_sch (KiCad schematic)
At the start: 25 parts, among them J1 MicroLab, J2 Pump 1, J3 Pump 2, Q1 NX7002BKR, Q2 NX7002BKR, Q3 NX7002BKR

Commit message: fin
Parts:
- added H1, H2, H3, H4: M2, MountingHole:MountingHole_2.2mm_M2_DIN965_Pad_TopOnly, symbol Mechanical:MountingHole_Pad
Connections:
- net GND: now also H1.1, H2.1, H3.1, H4.1
Changed lines of the file:
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@@
   (junction (at 205.74 114.3) (diameter 0) (color 0 0 0 0)
   )
+  (junction (at 58.674 154.94) (diameter 0) (color 0 0 0 0)
+  )
   (junction (at 190.5 81.28) (diameter 0) (color 0 0 0 0)
   )
+  (junction (at 62.23 154.94) (diameter 0) (color 0 0 0 0)
+  )
   (junction (at 149.86 68.58) (diameter 0) (color 0 0 0 0)
   )
@@
   (junction (at 132.08 144.78) (diameter 0) (color 0 0 0 0)
   )
+  (junction (at 66.04 154.94) (diameter 0) (color 0 0 0 0)
+  )
   (junction (at 185.42 114.3) (diameter 0) (color 0 0 0 0)
   )
@@
     (stroke (width 0) (type default) (color 0 0 0 0))
   )
+  (wire (pts (xy 58.674 154.94) (xy 62.23 154.94))
+    (stroke (width 0) (type default) (color 0 0 0 0))
+  )
   (wire (pts (xy 193.04 124.46) (xy 193.04 127))
     (stroke (width 0) (type default) (color 0 0 0 0))
@@
     (stroke (width 0) (type default) (color 0 0 0 0))
   )
+  (wire (pts (xy 62.23 154.94) (xy 62.23 157.48))
+    (stroke (width 0) (type default) (color 0 0 0 0))
+  )
   (wire (pts (xy 165.1 66.04) (xy 165.1 68.58))
     (stroke (width 0) (type default) (color 0 0 0 0))
@@
     (stroke (width 0) (type default) (color 0 0 0 0))
   )
+  (wire (pts (xy 58.674 152.4) (xy 58.674 154.94))
+    (stroke (width 0) (type default) (color 0 0 0 0))
+  )
   (wire (pts (xy 142.24 132.08) (xy 142.24 134.62))
     (stroke (width 0) (type default) (color 0 0 0 0))
@@
     (stroke (width 0) (type default) (color 0 0 0 0))
   )
+  (wire (pts (xy 62.23 154.94) (xy 66.04 154.94))
+    (stroke (width 0) (type default) (color 0 0 0 0))
+  )
   (wire (pts (xy 218.44 115.062) (xy 218.44 114.3))
     (stroke (width 0) (type default) (color 0 0 0 0))
@@
     (stroke (width 0) (type default) (color 0 0 0 0))
   )
+  (wire (pts (xy 50.8 154.94) (xy 58.674 154.94))
+    (stroke (width 0) (type default) (color 0 0 0 0))
+  )
+  (wire (pts (xy 66.04 152.4) (xy 66.04 154.94))
+    (stroke (width 0) (type default) (color 0 0 0 0))
+  )
   (wire (pts (xy 187.96 116.84) (xy 185.42 116.84))
     (stroke (width 0) (type default) (color 0 0 0 0))
@@
     (stroke (width 0) (type default) (color 0 0 0 0))
   )
+  (wire (pts (xy 73.66 154.94) (xy 73.66 152.4))
+    (stroke (width 0) (type default) (color 0 0 0 0))
+  )
   (wire (pts (xy 134.62 66.04) (xy 134.62 68.58))
     (stroke (width 0) (type default) (color 0 0 0 0))
@@
     (stroke (width 0) (type default) (color 0 0 0 0))
   )
+  (wire (pts (xy 66.04 154.94) (xy 73.66 154.94))
+    (stroke (width 0) (type default) (color 0 0 0 0))
+  )
   (wire (pts (xy 195.58 139.7) (xy 195.58 142.24))
     (stroke (width 0) (type default) (color 0 0 0 0))
@@
   )
   (wire (pts (xy 83.82 101.6) (xy 78.74 101.6))
+    (stroke (width 0) (type default) (color 0 0 0 0))
+  )
+  (wire (pts (xy 50.8 152.4) (xy 50.8 154.94))
     (stroke (width 0) (type default) (color 0 0 0 0))
   )
@@
     (pin "3")
   )
+  (symbol (lib_id "Mechanical:MountingHole_Pad") (at 73.66 149.86 0) (unit 1)
+    (in_bom yes) (on_board yes) (fields_autoplaced)
+    (property "Reference" "H4" (id 0) (at 76.2 147.7553 0)
+      (effects (font (size 1.27 1.27)) (justify left))
+    )
+    (property "Value" "M2" (id 1) (at 76.2 150.2922 0)
+      (effects (font (size 1.27 1.27)) (justify left))
+    )
+    (property "Footprint" "MountingHole:MountingHole_2.2mm_M2_DIN965_Pad_TopOnly" (id 2) (at 73.66 149.86 0)
+      (effects (font (size 1.27 1.27)) hide)
+    )
+    (property "Datasheet" "~" (id 3) (at 73.66 149.86 0)
+      (effects (font (size 1.27 1.27)) hide)
+    )
+    (pin "1")
+  )
   (symbol (lib_id "Device:LED_Small") (at 154.94 128.778 90) (unit 1)
     (in_bom yes) (on_board yes) (fields_autoplaced)
@@
     (pin "1")
     (pin "2")
+  )
+  (symbol (lib_id "power:GND") (at 62.23 157.48 0) (unit 1)
+    (in_bom yes) (on_board yes) (fields_autoplaced)
+    (property "Reference" "#PWR0112" (id 0) (at 62.23 163.83 0)
+      (effects (font (size 1.27 1.27)) hide)
+    )
+    (property "Value" "GND" (id 1) (at 62.23 161.9234 0))
+    (property "Footprint" "" (id 2) (at 62.23 157.48 0)
+      (effects (font (size 1.27 1.27)) hide)
+    )
+    (property "Datasheet" "" (id 3) (at 62.23 157.48 0)
+      (effects (font (size 1.27 1.27)) hide)
+    )
+    (pin "1")
+  )
+  (symbol (lib_id "Mechanical:MountingHole_Pad") (at 66.04 149.86 0) (unit 1)
+    (in_bom yes) (on_board yes) (fields_autoplaced)
+    (property "Reference" "H3" (id 0) (at 68.58 147.7553 0)
+      (effects (font (size 1.27 1.27)) (justify left))
+    )
+    (property "Value" "M2" (id 1) (at 68.58 150.2922 0)
+      (effects (font (size 1.27 1.27)) (justify left))
+    )
+    (property "Footprint" "MountingHole:MountingHole_2.2mm_M2_DIN965_Pad_TopOnly" (id 2) (at 66.04 149.86 0)
+      (effects (font (size 1.27 1.27)) hide)
+    )
+    (property "Datasheet" "~" (id 3) (at 66.04 149.86 0)
+      (effects (font (size 1.27 1.27)) hide)
+    )
+    (pin "1")
   )
   (symbol (lib_id "power:GND") (at 200.66 88.9 0) (unit 1)
@@
     (pin "1")
   )
+  (symbol (lib_id "Mechanical:MountingHole_Pad") (at 50.8 149.86 0) (unit 1)
+    (in_bom yes) (on_board yes) (fields_autoplaced)
+    (property "Reference" "H1" (id 0) (at 53.34 147.7553 0)
+      (effects (font (size 1.27 1.27)) (justify left))
+    )
+    (property "Value" "M2" (id 1) (at 53.34 150.2922 0)
+      (effects (font (size 1.27 1.27)) (justify left))
+    )
+    (property "Footprint" "MountingHole:MountingHole_2.2mm_M2_DIN965_Pad_TopOnly" (id 2) (at 50.8 149.86 0)
+      (effects (font (size 1.27 1.27)) hide)
+    )
+    (property "Datasheet" "~" (id 3) (at 50.8 149.86 0)
+      (effects (font (size 1.27 1.27)) hide)
+    )
+    (pin "1")
+  )
+  (symbol (lib_id "Mechanical:MountingHole_Pad") (at 58.674 149.86 0) (unit 1)
+    (in_bom yes) (on_board yes) (fields_autoplaced)
+    (property "Reference" "H2" (id 0) (at 61.214 147.7553 0)
+      (effects (font (size 1.27 1.27)) (justify left))
+    )
+    (property "Value" "M2" (id 1) (at 61.214 150.2922 0)
+      (effects (font (size 1.27 1.27)) (justify left))
+    )
+    (property "Footprint" "MountingHole:MountingHole_2.2mm_M2_DIN965_Pad_TopOnly" (id 2) (at 58.674 149.86 0)
+      (effects (font (size 1.27 1.27)) hide)
+    )
+    (property "Datasheet" "~" (id 3) (at 58.674 149.86 0)
+      (effects (font (size 1.27 1.27)) hide)
+    )
+    (pin "1")
+  )
   (sheet_instances
     (path "/" (page "1"))
@@
       (reference "#PWR0111") (unit 1) (value "GND") (footprint "")
     )
+    (path "/81b0081b-8b91-4528-8f66-1603526da330"
+      (reference "#PWR0112") (unit 1) (value "GND") (footprint "")
+    )
     (path "/19db885a-b711-4825-bf73-0e696d15cf61"
       (reference "D1") (unit 1) (value "158301250 ") (footprint "Mouser Parts:158301250")
@@
       (reference "D9") (unit 1) (value "Debug") (footprint "LED_SMD:LED_0402_1005Metric")
     )
+    (path "/ea2c131a-e4f0-4b3b-b7e4-71c3c2730e2b"
+      (reference "H1") (unit 1) (value "M2") (footprint "MountingHole:MountingHole_2.2mm_M2_DIN965_Pad_TopOnly")
+    )
+    (path "/f5fca380-6e47-434e-8021-4aa62e28b373"
+      (reference "H2") (unit 1) (value "M2") (footprint "MountingHole:MountingHole_2.2mm_M2_DIN965_Pad_TopOnly")
+    )
+    (path "/86c625bb-001a-4b78-94d1-a03ec1599995"
+      (reference "H3") (unit 1) (value "M2") (footprint "MountingHole:MountingHole_2.2mm_M2_DIN965_Pad_TopOnly")
+    )
+    (path "/32328943-0cda-4c14-bc4d-a633d495fa1e"
+      (reference "H4") (unit 1) (value "M2") (footprint "MountingHole:MountingHole_2.2mm_M2_DIN965_Pad_TopOnly")
+    )
     (path "/08da4816-0b0d-4c01-9e19-a88e27d5a270"

Commit message: goodnight
Parts:
- R1, R3, R4: value 180 -> 510
- R5, R8: value 240 -> 1k
Changed lines of the file:
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@@
       (effects (font (size 1.27 1.27)) (justify left))
     )
-    (property "Value" "240" (id 1) (at 202.1586 57.5822 0)
+    (property "Value" "1k" (id 1) (at 202.1586 57.5822 0)
       (effects (font (size 1.27 1.27)) (justify left))
     )
@@
       (effects (font (size 1.27 1.27)) (justify left))
     )
-    (property "Value" "180" (id 1) (at 151.3586 57.5822 0)
+    (property "Value" "510" (id 1) (at 151.3586 57.5822 0)
       (effects (font (size 1.27 1.27)) (justify left))
     )
@@
       (effects (font (size 1.27 1.27)) (justify left))
     )
-    (property "Value" "240" (id 1) (at 181.8386 57.5822 0)
+    (property "Value" "1k" (id 1) (at 181.8386 57.5822 0)
       (effects (font (size 1.27 1.27)) (justify left))
     )
@@
       (effects (font (size 1.27 1.27)) (justify left))
     )
-    (property "Value" "180" (id 1) (at 136.1186 57.5822 0)
+    (property "Value" "510" (id 1) (at 136.1186 57.5822 0)
       (effects (font (size 1.27 1.27)) (justify left))
     )
@@
       (effects (font (size 1.27 1.27)) (justify left))
     )
-    (property "Value" "180" (id 1) (at 166.5986 57.5822 0)
+    (property "Value" "510" (id 1) (at 166.5986 57.5822 0)
       (effects (font (size 1.27 1.27)) (justify left))
     )
@@
     )
     (path "/c8c171de-6a1e-4dca-893c-23f8fbd340f2"
-      (reference "R1") (unit 1) (value "180") (footprint "Resistor_SMD:R_0402_1005Metric")
+      (reference "R1") (unit 1) (value "510") (footprint "Resistor_SMD:R_0402_1005Metric")
     )
     (path "/b4ef17f7-3a18-41b6-90bb-9bb93af9173c"
@@
     )
     (path "/78db8bb1-d96a-463d-9b03-b7208234a9ac"
-      (reference "R3") (unit 1) (value "180") (footprint "Resistor_SMD:R_0402_1005Metric")
+      (reference "R3") (unit 1) (value "510") (footprint "Resistor_SMD:R_0402_1005Metric")
     )
     (path "/cd35a060-201d-4948-9fc5-44229ffda806"
-      (reference "R4") (unit 1) (value "180") (footprint "Resistor_SMD:R_0402_1005Metric")
+      (reference "R4") (unit 1) (value "510") (footprint "Resistor_SMD:R_0402_1005Metric")
     )
     (path "/ae95ab19-3c33-4535-9d78-ecf6bd090dcb"
-      (reference "R5") (unit 1) (value "240") (footprint "Resistor_SMD:R_0402_1005Metric")
+      (reference "R5") (unit 1) (value "1k") (footprint "Resistor_SMD:R_0402_1005Metric")
     )
     (path "/54a6fbfa-fa24-4ec6-9fed-b1b8715ac6ed"
@@
     )
     (path "/539c8975-706b-4c46-84f4-c5743bffc3d4"
-      (reference "R8") (unit 1) (value "240") (footprint "Resistor_SMD:R_0402_1005Metric")
+      (reference "R8") (unit 1) (value "1k") (footprint "Resistor_SMD:R_0402_1005Metric")
     )
     (path "/dcb8a0d6-b775-43b9-9514-ed3c4ab90f2c"
