File: pcb/pcb_rear/pcb_rear.kicad_pcb (KiCad board)
At the start: 2 copper layers, 23 parts, among them J1 MicroLab Input, J2 Pump, J3 DFRobot O2, J4 DFRobot NH3, Q1 T2N7002AK, Q2 T2N7002AK, Q3 T2N7002AK, Q4 T2N7002AK, U1 USEQGSE CO2, U2 USEQGSE CH4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

Commit message: fin
Parts:
- removed Q2, Q3, Q4: T2N7002AK, Package_TO_SOT_SMD:SOT-23
- removed U3, U4: XC9265A331MR-G, SamacSys:SOT95P280X130-5N
- added C3: 0.1uF, Capacitor_SMD:C_0402_1005Metric, F.Cu at (-0.50, 15.7)
- added C4: 10uF, Capacitor_SMD:C_0402_1005Metric, F.Cu at (-2.50, 9.85)
- added C5: 0.1uF, Capacitor_SMD:C_0402_1005Metric, F.Cu at (0.50, 17.6)
- added C6: 0.1uF, Capacitor_SMD:C_0402_1005Metric, F.Cu at (0.50, 15.7)
- added C7: 0.1uF, Capacitor_SMD:C_0402_1005Metric, F.Cu at (7.00, 15.2)
- added C8: 10uF, Capacitor_SMD:C_0402_1005Metric, F.Cu at (5.20, 9.85)
- added D2: D_Small, Diode_SMD:D_SOD-323, F.Cu at (3.00, 22.8)
- added D3: PWR, LED_SMD:LED_0402_1005Metric, F.Cu at (-4.85, 9.85)
- added G***: LOGO, LOGO, B.Cu at (-0.50, 3.60)
- added H1: M2, MountingHole:MountingHole_2.2mm_M2_DIN965_Pad, F.Cu at (-8.60, 12.4)
- added H2: M2, MountingHole:MountingHole_2.2mm_M2_DIN965_Pad, F.Cu at (8.60, 12.4)
- added H3: M2, MountingHole:MountingHole_2.2mm_M2_DIN965_Pad, F.Cu at (8.60, 27.8)
- added H4: M2, MountingHole:MountingHole_2.2mm_M2_DIN965_Pad, F.Cu at (-8.60, 27.8)
- added J5: Fan, Connector_JST:JST_SH_BM02B-SRSS-TB_1x02-1MP_P1.00mm_Vertical, F.Cu at (8.10, 22.6)
- added J8: MEM2051-00-195-00-A, SamacSys:MEM20510019500A, F.Cu at (0.00, 0.00)
- added R9: 500, Resistor_SMD:R_0402_1005Metric, F.Cu at (-3.65, 9.85)
- C1, C2: value 100nF -> 0.1uF; footprint Capacitor_SMD:C_0603_1608Metric -> Capacitor_SMD:C_0402_1005Metric
- D1: footprint Diode_SMD:D_0603_1608Metric -> Diode_SMD:D_SOD-323
- J1: value MicroLab Input -> XIAO_L; footprint Connector_PinSocket_2.54mm:PinSocket_2x06_P2.54mm_Vertical -> Connector_PinSocket_2.54mm:PinSocket_1x07_P2.54mm_Vertical
- J2: value Pump -> XIAO_R; footprint Connector_PinSocket_2.54mm:PinSocket_1x02_P2.54mm_Vertical -> Connector_PinSocket_2.54mm:PinSocket_1x07_P2.54mm_Vertical
- J3: value DFRobot O2 -> MicroLab; footprint Connector_PinSocket_2.54mm:PinSocket_1x04_P2.54mm_Vertical -> Connector_JST:JST_SH_BM04B-SRSS-TB_1x04-1MP_P1.00mm_Vertical
- J4: value DFRobot NH3 -> O2 Sensor; footprint Connector_PinSocket_2.54mm:PinSocket_1x04_P2.54mm_Vertical -> Connector_JST:JST_SH_BM04B-SRSS-TB_1x04-1MP_P1.00mm_Vertical
- Q1: value T2N7002AK -> NX7002BKR
- R1, R2, R3, R4, R5: value 10k -> 50k; footprint Resistor_SMD:R_0603_1608Metric -> Resistor_SMD:R_0402_1005Metric
- R6, R7, R8: footprint Resistor_SMD:R_0603_1608Metric -> Resistor_SMD:R_0402_1005Metric
- moved R3 187.2 mm to (1.30, 9.85), turned to -90 degrees
- moved R4 187.1 mm to (0.00, 9.85), turned to 90 degrees
- moved R2 187.0 mm to (2.60, 9.85), turned to 90 degrees
- moved R5 186.5 mm to (-1.30, 9.85), turned to 90 degrees
- moved R1 184.8 mm to (3.90, 9.85), turned to 90 degrees
- moved C2 183.6 mm to (-7.00, 16.4)
- moved D1 183.4 mm to (-3.00, 22.8), turned to 90 degrees
- moved C1 182.9 mm to (-7.00, 15.2)
- moved R6 181.3 mm to (-5.70, 26.5), turned to -90 degrees
- moved J2 180.4 mm to (9.40, -7.60)
- moved J1 179.6 mm to (-9.40, -7.62)
- moved R8 179.3 mm to (4.50, 26.5), turned to 90 degrees
- moved R7 179.2 mm to (-4.50, 26.5), turned to -90 degrees
- moved Q1 176.4 mm to (0.00, 22.8), turned to 180 degrees
- moved U1 173.9 mm to (-3.40, 17.1)
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Connections:
- C1 pad 2: Net-(C1-Pad2) -> +3.3V
- C2 pad 2: Net-(U2-Pad3) -> Net-(C2-Pad2)
- D1 pad 1: /V_PUMP -> Net-(D1-Pad1)
- D1 pad 2: GND -> +5V
- J1 pad 1: /SDA -> +5V
- J1 pad 2: unconnected-(J1-Pad2) -> GND
- J1 pad 3: /SCL -> +3.3V
- J1 pad 4: /V_O2 -> /MOSI
- J1 pad 5: VCC -> /MISO
- J1 pad 6: /V_NH3 -> /SCK
- J1 pad 7: GND -> /TX
- J2 pad 1: /V_PUMP -> /D0
- J2 pad 2: GND -> /D1
- J3 pad 1: /SDA -> Net-(D1-Pad1)
- J3 pad 2: /SCL -> /RX
- J3 pad 3: GND -> /TX
- J3 pad 4: /V_O2 -> GND
- J4 pad 1: /SDA -> +3.3V
- J4 pad 2: /SCL -> GND
- J4 pad 3: GND -> /SDA
- J4 pad 4: /V_NH3 -> /SCL
- Q1 pad 1: /V_CO2 -> /D1
- Q1 pad 2: Net-(R1-Pad2) -> GND
- Q1 pad 3: /SDA -> Net-(D2-Pad2)
- R1 pad 1: /V_CO2 -> +3.3V
- R1 pad 2: Net-(R1-Pad2) -> Net-(J8-PadP1)
- R2 pad 1: VCC -> +3.3V
- R2 pad 2: /SDA -> /D0
- R3 pad 1: Net-(R3-Pad1) -> +3.3V
- R3 pad 2: /V_CO2 -> /MOSI
- R4 pad 1: /SCL -> +3.3V
- R4 pad 2: VCC -> /MISO
- R5 pad 1: /V_CH4 -> +3.3V
- R5 pad 2: Net-(U2-Pad26) -> Net-(J8-PadP8)
- R6 pad 1: VCC -> /SDA
- R6 pad 2: /SDA -> +3.3V
- R7 pad 1: Net-(U2-Pad37) -> /SCL
- R7 pad 2: /V_CH4 -> +3.3V
- R8 pad 1: /SCL -> GND
- R8 pad 2: VCC -> /D1
- U1 pad 1: /V_CO2 -> +3.3V
- U1 pad 23: /V_CO2 -> +3.3V
- U1 pad 25: /CO2_INT -> unconnected-(U1-Pad25)
- U1 pad 26: Net-(R1-Pad2) -> /SDA
- U1 pad 27: (no net) -> /SCL
- U1 pad 3: Net-(C1-Pad2) -> Net-(C2-Pad2)
- U2 pad 1: /V_CH4 -> +3.3V
- U2 pad 23: /V_CH4 -> +3.3V
- U2 pad 25: /CH4_INT -> unconnected-(U2-Pad25)
- U2 pad 26: Net-(U2-Pad26) -> /SDA
- U2 pad 27: (no net) -> /SCL
- U2 pad 3: Net-(U2-Pad3) -> Net-(C5-Pad2)
Routing:
- net +3.3V: track 0.00 -> 69.3 mm, vias 0 -> 1
- net /SCL: track 0.00 -> 51.4 mm, vias 0 -> 2
- net +5V: track 0.00 -> 45.7 mm, vias 0 -> 2
- net /D1: track 0.00 -> 45.7 mm
- net /SDA: track 0.00 -> 45.6 mm, vias 0 -> 3
- net /RX: track 0.00 -> 26.5 mm, vias 0 -> 1
- net /TX: track 0.00 -> 26.2 mm, vias 0 -> 1
- net /D0: track 0.00 -> 24.5 mm
- net /MISO: track 0.00 -> 21.6 mm
- net /MOSI: track 0.00 -> 20.3 mm
- net Net-(D2-Pad2): track 0.00 -> 15.8 mm
- net /SCK: track 0.00 -> 9.75 mm
- net Net-(J8-PadP8): track 0.00 -> 8.35 mm
- net Net-(J8-PadP1): track 0.00 -> 6.50 mm
- net Net-(D1-Pad1): track 0.00 -> 6.37 mm
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- added copper zone on B.Cu, net GND
- added copper zone on F.Cu, net GND
Other:
- board outline added: 21.6 x 39 mm
- board text added: "JLCJLCJLCJLC"
- board text added: "SAS SpaceLab 2023"

Commit message: goodnight
Parts:
- turned D1 to -90 degrees
Connections:
- D1 pad 1: Net-(D1-Pad1) -> +5V
- D1 pad 2: +5V -> Net-(D1-Pad2)
- J3 pad 1: Net-(D1-Pad1) -> Net-(D1-Pad2)
Routing:
- net Net-(D1-Pad2): track 0.00 -> 6.37 mm
- net Net-(D1-Pad1): track 6.37 -> 0.00 mm
Other:
- board text added: "Fan"
- board text added: "ML"
- board text added: "O2"
Changed lines of the file:
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@@
   (net 22 "/RX")
   (net 23 "Net-(C5-Pad2)")
-  (net 24 "Net-(D1-Pad1)")
+  (net 24 "Net-(D1-Pad2)")
   (net 25 "Net-(J8-PadP1)")
   (net 26 "Net-(J8-PadP8)")
-  (net 27 "Net-(R9-Pad1)")
+  (net 27 "Net-(D3-Pad2)")
   (footprint "MountingHole:MountingHole_2.2mm_M2_DIN965_Pad" (layer "F.Cu")
     (at -8.6 12.4)
@@
       (net 1 "GND") (pinfunction "K") (pintype "passive"))
     (pad "2" smd roundrect (at 0.485 0 270) (size 0.59 0.64) (layers "F.Cu" "F.Paste" "F.Mask") (roundrect_rratio 0.25)
-      (net 27 "Net-(R9-Pad1)") (pinfunction "A") (pintype "passive"))
+      (net 27 "Net-(D3-Pad2)") (pinfunction "A") (pintype "passive"))
     (model "${KICAD6_3DMODEL_DIR}/LED_SMD.3dshapes/LED_0402_1005Metric.wrl"
       (offset (xyz 0 0 0))
@@
     (fp_line (start 3 1) (end 3 -1.9) (layer "F.Fab") (width 0.1))
     (pad "1" smd roundrect (at -1.5 1.325 180) (size 0.6 1.55) (layers "F.Cu" "F.Paste" "F.Mask") (roundrect_rratio 0.25)
-      (net 24 "Net-(D1-Pad1)") (pinfunction "Pin_1") (pintype "passive"))
+      (net 24 "Net-(D1-Pad2)") (pinfunction "Pin_1") (pintype "passive"))
     (pad "2" smd roundrect (at -0.5 1.325 180) (size 0.6 1.55) (layers "F.Cu" "F.Paste" "F.Mask") (roundrect_rratio 0.25)
       (net 22 "/RX") (pinfunction "Pin_2") (pintype "passive"))
@@
   )
   (footprint "Diode_SMD:D_SOD-323" (layer "F.Cu")
-    (at -3 22.8 90)
+    (at -3 22.8 -90)
     (descr "SOD-323")
     (tags "SOD-323")
@@
     (property "Sheetname" "")
     (attr smd)
-    (fp_text reference "D1" (at 0 -1.7 90 unlocked) (layer "F.SilkS")
+    (fp_text reference "D1" (at 0 1.6 90 unlocked) (layer "F.SilkS")
       (effects (font (size 0.8 0.8) (thickness 0.15)))
     )
@@
     (fp_line (start -0.3 0) (end -0.5 0) (layer "F.Fab") (width 0.1))
     (fp_line (start -0.9 0.7) (end -0.9 -0.7) (layer "F.Fab") (width 0.1))
-    (pad "1" smd rect (at -1.05 0 90) (size 0.6 0.45) (layers "F.Cu" "F.Paste" "F.Mask")
-      (net 24 "Net-(D1-Pad1)") (pinfunction "K") (pintype "passive"))
-    (pad "2" smd rect (at 1.05 0 90) (size 0.6 0.45) (layers "F.Cu" "F.Paste" "F.Mask")
-      (net 4 "+5V") (pinfunction "A") (pintype "passive"))
+    (pad "1" smd rect (at -1.05 0 270) (size 0.6 0.45) (layers "F.Cu" "F.Paste" "F.Mask")
+      (net 4 "+5V") (pinfunction "K") (pintype "passive"))
+    (pad "2" smd rect (at 1.05 0 270) (size 0.6 0.45) (layers "F.Cu" "F.Paste" "F.Mask")
+      (net 24 "Net-(D1-Pad2)") (pinfunction "A") (pintype "passive"))
     (model "${KICAD6_3DMODEL_DIR}/Diode_SMD.3dshapes/D_SOD-323.wrl"
       (offset (xyz 0 0 0))
@@
     (fp_line (start -0.525 -0.27) (end 0.525 -0.27) (layer "F.Fab") (width 0.1))
     (pad "1" smd roundrect (at -0.51 0 90) (size 0.54 0.64) (layers "F.Cu" "F.Paste" "F.Mask") (roundrect_rratio 0.25)
-      (net 27 "Net-(R9-Pad1)") (pintype "passive"))
+      (net 27 "Net-(D3-Pad2)") (pintype "passive"))
     (pad "2" smd roundrect (at 0.51 0 90) (size 0.54 0.64) (layers "F.Cu" "F.Paste" "F.Mask") (roundrect_rratio 0.25)
       (net 4 "+5V") (pintype "passive"))
@@
     (effects (font (size 0.8 0.8) (thickness 0.15)))
   )
+  (gr_text "ML" (at -3 25.6) (layer "F.SilkS")
+    (effects (font (size 0.8 0.8) (thickness 0.15)))
+  )
+  (gr_text "Fan" (at 6.3 24.8 90) (layer "F.SilkS")
+    (effects (font (size 0.8 0.8) (thickness 0.15)))
+  )
+  (gr_text "O2" (at -6.4 18.7 270) (layer "F.SilkS")
+    (effects (font (size 0.8 0.8) (thickness 0.15)))
+  )
